File: KiCAD/MC6803EP-SBC6809E.kicad_sch (KiCad schematic)
At the start: 10 parts, among them U1 MC6809E ソケット, U2 74HCT02

Commit message: REV1 ガーバーデータ出力
Parts:
- added R1, R2, R3: 10k, Resistor_THT:R_Axial_DIN0207_L6.3mm_D2.5mm_P10.16mm_Horizontal, symbol Device:R_Small_US
- J1: value (none) -> I/O PIN; footprint (none) -> Connector_PinHeader_2.54mm:PinHeader_1x08_P2.54mm_Horizontal
- J2: value (none) -> CONT PIN; footprint (none) -> Connector_PinHeader_2.54mm:PinHeader_1x05_P2.54mm_Horizontal
- J3: value (none) -> SBC68_BUS; footprint (none) -> Connector_PinHeader_2.54mm:PinHeader_2x20_P2.54mm_Horizontal
- U1: footprint Package_DIP:DIP-40_W15.24mm_Socket_LongPads -> (none)
- U2: footprint Package_DIP:DIP-14_W7.62mm_Socket_LongPads -> (none)
- U3: value (none) -> MC6803EP
- U4: value (none) -> 74LS573
Connections:
- net GND: now also R2.2, R3.2
- net VCC: now also R1.1
- net at J2.3 (Pin_3), U3.10 (SCLK-P22): now also R2.1
- net at J2.1 (Pin_1), U3.8 (TIN-P20): now also R3.1
- net at J2.2 (Pin_2), U3.9 (T-OUT-P21): now also R1.2
Other:
- moved on the sheet: U2A, U2B, U2C, U2D

Commit message: REV1 回路変更(シリアル端子)、ガーバー再出力
Parts:
- removed J2: CONT PIN, Connector_PinHeader_2.54mm:PinHeader_1x05_P2.54mm_Horizontal, symbol Connector_Generic:Conn_01x05
- added J2: SERIAL Con, Connector_PinHeader_2.54mm:PinHeader_1x06_P2.54mm_Horizontal, symbol Connector_Generic:Conn_01x06
- U1, U3: footprint (none) -> Package_DIP:DIP-40_W15.24mm_Socket
- U2: footprint (none) -> Package_DIP:DIP-14_W7.62mm_Socket
- U4: footprint (none) -> Package_DIP:DIP-20_W7.62mm_Socket
Connections:
- net GND: now also J2.1 (Pin_1)
- net at U3.11 (RDATA-P23): now also J2.4 (Pin_4)
- net at U3.12 (TDATA-P24): now also J2.5 (Pin_5)
- no-connect marks 18 -> 21
Other:
- note added: "+5V"
- note added: "CTS"
- note added: "GND"
- note added: "RTS"
- note added: "RxD"
- note added: "TxD"
